File: h9ps.kicad_pcb (KiCad board)
At the start: 2 copper layers, 70 x 60 mm, 76 parts, among them J1 AVR-ISP-6, J2 Conn_01x03, J3 DB9, J4 Conn_01x04, Q1 2N7002, Q2 BSS84, Q3 2N7002, Q4 2N7002, U1 TLC272, U2 MCP1541-TT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

Commit message: fix, v1.0
Parts:
-  : renamed from REF**
- D3: moved to F.Cu
- V out: renamed from H2
- renumbered H1 to V+, H3 to V-
Routing:
- net +5V: track 108.3 -> 115.0 mm
- net GND: track 23.3 -> 18.4 mm
